File: Pure Sequencer.sch (EAGLE design)
At the start: 132 parts, among them Q1 20MHz, T1 2N3904, T2 2N3904, U1 ATMEGA328P, U2 QUAD_OPAMP, U3 QUAD_OPAMP, U4 4051, U5 7805, U6 QUAD_OPAMP

Commit message: Sequencer 2.2
Parts:
- removed C11, C13, C15, C17, C19, C21, C23, C25, C8: *, rcl:C-USC0805K
- removed C9: 47p, rcl:C-USC0805K
- removed GLIDE1: rate, INSTRUO:Q-POT
- removed U$7: PB6149L-5, INSTRUO:PB6149L-5
- removed U1: ATMEGA328P, SparkFun-DigitalIC:ATMEGA328_SMT
- removed U2, U3, U6: QUAD_OPAMP, INSTRUO:QUAD_OPAMP
- removed U4: 4051, INSTRUO:MUX!
- removed U5: 7805, INSTRUO:V-REG
- added D10, D3, D4, D5, D6, D7, D8, D9: 1N914, GMSN:DIODEDO-41
- added IC1: BA178M05FP, GMSN:VOLTAGE_REG_POS05DT
- added IC2, IC3, IC4: TL074, GMSN:OPAMP_QUADD
- added IC5: ATMEGA328P, GMSN:MICROPROCESSOR_ATMEGA328_SMT
- added IC6: CD4051, GMSN:MUX_1X8_CD4051
- added R60: 200k, GMSN:RESISTOR_USR0805
- added R61: 100k, GMSN:RESISTOR_USR0805
- added RANGE: SWITCH_TOGGLE, GMSN:SWITCH_TOGGLE
- added RATE: B100k, GMSN:RESISTOR_VARIABLE9MM_POT
- added SW1: (no value), GMSN:SWITCH_PUSHBUTTON_LED
- added TR1: 100k, GMSN:RESISTOR_VARIABLETRIMMER_TH
- C1, C2: value 22p -> 22pF; device rcl:C-USC0805K -> GMSN:CAPACITOR-USC0805
- C10, C12, C14, C16, C18, C20, C22, C24: value 47p -> 100pF; device rcl:C-USC0805K -> GMSN:CAPACITOR-USC0805
- C26, C4, C5: value 10u -> 10uF; device rcl:CPOL-US153CLV-0505 -> GMSN:CAPACITOR_POL-US153CLV-0505
- C27, C28, C29, C30, C31, C32, C33, C34, C35, C36: value 0.1u -> 100nF; device rcl:C-USC0805K -> GMSN:CAPACITOR-USC0805
- C3: device rcl:C-USC0805K -> GMSN:CAPACITOR-USC0805
- C6, C7: value 47p -> 47pF; device rcl:C-USC0805K -> GMSN:CAPACITOR-USC0805
- CLK_IN, CLOCK_OUT, CV_OUT, GATE1, GATE2, GATE3, GATE4, GATE5, GATE6, GATE7, GATE8, RESET: value S_JACK -> PJ301M-12; device INSTRUO:S_JACK -> GMSN:SOCKET_MONO_3.5MMPJ301M-12
- D1, D2: value (none) -> STTH102A; device adafruit:DIODESMA -> GMSN:DIODESMA
- DIRSW: value TOGGLE_ON_OFF_ON -> SWITCH_TOGGLE; device INSTRUO:TOGGLE_ON_OFF_ON -> GMSN:SWITCH_TOGGLE
- FADER1, FADER2, FADER3, FADER4, FADER5, FADER6, FADER7, FADER8: value LED_FADER -> 100k; device INSTRUO:LED_FADER -> GMSN:RESISTOR_VARIABLE_LED
- GLIDE: value B100K -> B100k; device INSTRUO:Q-POT -> GMSN:RESISTOR_VARIABLE9MM_POT
- ISP1: value AVRISP-6 -> HEADER2X3-6; device adafruit:AVRISP-6 -> GMSN:HEADER2X3-6
- JP1: value M05X2SHD -> HEADER2X5SHD; device SparkFun-Connectors:M05X2SHD -> GMSN:HEADER2X5SHD
- Q1: device adafruit:CRYSTALHC49UP -> GMSN:CRYSTALHC49UP
- R1: value 200R -> 0R; device rcl:R-US_R0805 -> GMSN:RESISTOR_USR0805
- R10, R15, R20, R25, R30, R35, R40, R45, R50, R56, R7: device rcl:R-US_R0805 -> GMSN:RESISTOR_USR0805
- R11, R12, R16, R17, R19, R21, R22, R24, R26, R27, R29, R31, R32, R34, R36, R37, R39, R41, R42, R44, R46, R47, R49, R51, R52, R54, R55, R58, R59, R6, R9: value 100K -> 100k; device rcl:R-US_R0805 -> GMSN:RESISTOR_USR0805
- R13, R14, R18, R23, R28, R33, R38, R43, R48, R53, R57: value 1K -> 1k; device rcl:R-US_R0805 -> GMSN:RESISTOR_USR0805
- R2: value 30K -> 34k; device rcl:R-US_R0805 -> GMSN:RESISTOR_USR0805
- R3: value 50K -> 56k; device rcl:R-US_R0805 -> GMSN:RESISTOR_USR0805
- R4: value 1K -> 0R; device rcl:R-US_R0805 -> GMSN:RESISTOR_USR0805
- R5, R8: value 10K -> 10k; device rcl:R-US_R0805 -> GMSN:RESISTOR_USR0805
- T1, T2: value 2N3904 -> MMBT3904; device INSTRUO:TRANSISTOR_MMBT3904 -> GMSN:TRANSISTOR_NPNSOT23
Connections:
- removed net +5V: C26.+, C33.1, C34.1, C35.1, C36.1, FADER1G$1.1, FADER2G$1.1, FADER3G$1.1, FADER4G$1.1, FADER5G$1.1, FADER6G$1.1, FADER7G$1.1, FADER8G$1.1, GLIDE1.1, ISP1.VCC, R5.2, R57.1, R8.2, U$7G$1.2, U$7G$1.4, U1.AVCC, U1.VCC@1, U1.VCC@2, U4.VCC, U5.OUT
- removed net MISO: ISP1.MISO, U1.PB4(MISO), U4.S1
- removed net MOSI: ISP1.MOSI, U1.PB3(MOSI/OC2), U4.S0
- removed net SCK: ISP1.SCK, U1.PB5(SCK), U4.S2
- new net 5V: C26.+, C33.1, C34.1, C35.1, C36.1, FADER1G$1.1, FADER2G$1.1, FADER3G$1.1, FADER4G$1.1, FADER5G$1.1, FADER6G$1.1, FADER7G$1.1, FADER8G$1.1, IC1.VO, IC5.AVCC, IC5.VCC@1, IC5.VCC@2, IC6.VCC, ISP1.VCC, R5.2, R57.1, R8.2, RATE.1, SW1G$1.2, SW1G$1.4
- new net A: IC5.PB3(MOSI/OC2), IC6.S0, ISP1.MOSI
- new net B: IC5.PB4(MISO), IC6.S1, ISP1.MISO
- new net C: IC5.PB5(SCK), IC6.S2, ISP1.SCK
- new net N$69: IC6.Z, R60.2
- new net N$70: RANGE.P, TR1.2, TR1.3
- new net N$71: D6.C, GATE4.TIP
- new net N$72: D5.C, GATE3.TIP
- new net N$73: D4.C, GATE2.TIP
- new net N$74: D3.C, GATE1.TIP
- new net N$75: D10.C, GATE8.TIP
- new net N$76: D9.C, GATE7.TIP
- new net N$77: D8.C, GATE6.TIP
- new net N$78: D7.C, GATE5.TIP
- net +12V: now also IC1.VI, IC2P.V+, IC3P.V+, IC4P.V+; no longer U2G$5.+12V, U3G$5.+12V, U5.IN, U6G$5.+12V
- net -12V: now also IC2P.V-, IC3P.V-, IC4P.V-; no longer U2G$6.-12V, U3G$6.-12V, U6G$6.-12V
- net CLK_IN: now also IC5.PD2(INT0); no longer U1.PD2(INT0)
- net CLK_OUT: now also IC2C.+IN, IC5.PB2(SS/OC1B); no longer U1.PB2(SS/OC1B), U6G$2.+IN, U6G$3.+IN
- net G0: now also IC3A.+IN, IC5.PC0(ADC0); no longer U1.PC0(ADC0), U2G$1.+IN
- net G1: now also IC3B.+IN, IC5.PC1(ADC1); no longer U1.PC1(ADC1), U2G$2.+IN
- net G2: now also IC3C.+IN, IC5.PC2(ADC2); no longer U1.PC2(ADC2), U2G$3.+IN
- net G3: now also IC3D.+IN, IC5.PC3(ADC3); no longer U1.PC3(ADC3), U2G$4.+IN
- net G4: now also IC4A.+IN, IC5.PC4(ADC4/SDA); no longer U1.PC4(ADC4/SDA), U3G$1.+IN
- net G5: now also IC4B.+IN, IC5.PC5(ADC5/SCL); no longer U1.PC5(ADC5/SCL), U3G$2.+IN
- net G6: now also IC4C.+IN, IC5.PB0(ICP); no longer U1.PB0(ICP), U3G$3.+IN
- net G7: now also IC4D.+IN, IC5.PB1(OC1A); no longer U1.PB1(OC1A), U3G$4.+IN
- net GND: now also CLK_IN.SLEEVE, CLOCK_OUT.SLEEVE, CV_OUT.SLEEVE, GATE1.SLEEVE, GATE2.SLEEVE, GATE3.SLEEVE, GATE4.SLEEVE, GATE5.SLEEVE, GATE6.SLEEVE, GATE7.SLEEVE, GATE8.SLEEVE, IC1.GND, IC5.AGND, IC5.GND@1, IC5.GND@2, IC6.E, IC6.GND, IC6.VEE, RANGE.S, RATE.3, RESET.SLEEVE; no longer C11.2, C13.2, C15.2, C17.2, C19.2, C21.2, C23.2, C25.2, C8.2, CLK_IN.GND, CLOCK_OUT.GND, CV_OUT.GND, GATE1.GND, GATE2.GND, GATE3.GND, GATE4.GND, GATE5.GND, GATE6.GND, GATE7.GND, GATE8.GND, GLIDE1.3, RESET.GND, U1.AGND, U1.GND@1, U1.GND@2, U4.E, U4.GND, U4.VEE, U5.GND
- net N$1: now also IC5.PB6(XTAL1/TOSC1); no longer U1.PB6(XTAL1/TOSC1)
- net N$11: now also IC6.Y4; no longer U4.Y4
- net N$12: now also IC6.Y3; no longer U4.Y3
- net N$13: now also IC6.Y2; no longer U4.Y2
- net N$14: now also IC6.Y1; no longer U4.Y1
- net N$15: now also IC6.Y0; no longer U4.Y0
- net N$16: now also IC2A.+IN; no longer U6G$1.+IN
- net N$18: now also IC2B.+IN, R61.2; no longer CLK_IN.TIP, R6.2
- net N$19: now also IC2A.-IN; no longer U6G$1.-IN
- net N$2: now also IC5.PB7(XTAL2/TOSC2); no longer U1.PB7(XTAL2/TOSC2)
- net N$20: now also IC2A.OUT; no longer U6G$1.OUT
- net N$24: now also IC2C.-IN; no longer C8.1, U6G$3.-IN
- net N$25: now also IC2C.OUT; no longer U6G$3.OUT
- net N$26: now also CLK_IN.TIP, R6.2, R61.1; no longer CLOCK_OUT.TIP, R11.1, R13.1
- net N$27: now also IC2B.-IN, IC2B.OUT, R14.2; no longer C9.1, U6G$2.-IN
- net N$28: now also CLOCK_OUT.TIP, R14.1; no longer C9.2, R14.2, U6G$2.OUT
- net N$29: now also CLK_IN.SWITCH, R11.1, R13.1; no longer CLK_IN.NORM, R14.1
- net N$3: now also IC2D.+IN, R60.1, TR1.1; no longer U4.Z, U6G$4.+IN
- net N$30: now also IC5.ADC7, RATE.2; no longer GLIDE1.2, U1.ADC7
- net N$32: now also IC3A.-IN; no longer C11.1, U2G$1.-IN
- net N$33: now also IC3A.OUT; no longer U2G$1.OUT
- net N$34: now also D3.A; no longer GATE1.TIP
- net N$37: now also IC3B.-IN; no longer C13.1, U2G$2.-IN
- net N$38: now also IC3B.OUT; no longer U2G$2.OUT
- net N$39: now also D4.A; no longer GATE2.TIP
- net N$4: now also IC2D.-IN, IC2D.OUT; no longer U6G$4.-IN, U6G$4.OUT
- net N$40: now also IC3C.-IN; no longer C15.1, U2G$3.-IN
- net N$41: now also IC3C.OUT; no longer U2G$3.OUT
- net N$42: now also D5.A; no longer GATE3.TIP
- net N$44: now also IC3D.-IN; no longer C17.1, U2G$4.-IN
- net N$45: now also IC3D.OUT; no longer U2G$4.OUT
- net N$46: now also D6.A; no longer GATE4.TIP
- net N$48: now also IC4A.-IN; no longer C19.1, U3G$1.-IN
- net N$49: now also IC4A.OUT; no longer U3G$1.OUT
- net N$50: now also D7.A; no longer GATE5.TIP
- net N$52: now also IC4B.-IN; no longer C21.1, U3G$2.-IN
- net N$53: now also IC4B.OUT; no longer U3G$2.OUT
- net N$54: now also D8.A; no longer GATE6.TIP
- net N$56: now also IC4C.-IN; no longer C23.1, U3G$3.-IN
- net N$57: now also IC4C.OUT; no longer U3G$3.OUT
- net N$58: now also D9.A; no longer GATE7.TIP
- net N$6: now also IC6.Y7; no longer U4.Y7
- net N$60: now also IC4D.-IN; no longer C25.1, U3G$4.-IN
- net N$61: now also IC4D.OUT; no longer U3G$4.OUT
- net N$62: now also D10.A; no longer GATE8.TIP
- net N$63: now also IC5.PD4(XCK/T0), SW1G$1.1, SW1G$1.3; no longer U$7G$1.1, U$7G$1.3, U1.PD4(XCK/T0)
- net N$64: now also IC5.PD5(T1), SW1G$2.A; no longer U$7G$2.A, U1.PD5(T1)
- net N$65: now also SW1G$2.C; no longer U$7G$2.C
- net N$67: now also IC5.PD6(AIN0); no longer U1.PD6(AIN0)
- net N$68: now also IC5.PD7(AIN1); no longer U1.PD7(AIN1)
- net N$7: now also IC6.Y6; no longer U4.Y6
- net N$8: now also IC6.Y5; no longer U4.Y5
- net RESET: now also IC5.PD3(INT1); no longer U1.PD3(INT1)
- net RST: now also IC5.PC6(/RESET); no longer U1.PC6(/RESET)
Other:
- moved on the sheet: R5, R6, R7

Commit message: Sequencer 2.3
Sequencer Updated to V2.3 20/4/21

Power Supply updated pull 5V from main case power supply, in line with low noise techniques.
Some resistor values reduced to 10k, in line with low noise techniques.
Traces rerouted.
Parts:
- removed IC1: BA178M05FP, GMSN:VOLTAGE_REG_POS05DT
- removed JP1: HEADER2X5SHD, GMSN:HEADER2X5SHD
- removed TR1: 100k, GMSN:RESISTOR_VARIABLETRIMMER_TH
- added JP2: HEADER2X8, GMSN:HEADER2X8
- added R62: 50k, GMSN:RESISTOR_USR0805
- R1: value 0R -> 100R
- R16, R17, R21, R22, R26, R27, R31, R32, R36, R37, R41, R42, R46, R47, R51, R52: value 100k -> 10k
- R4: value 0R -> 1k
Connections:
- removed net N$10: D2.C, JP1.1, JP1.2
- new net GALL: IC5.ADC6
- new net N$79: D2.C, JP2.1, JP2.2
- new net N$81: JP2.13, JP2.14
- new net N$82: JP2.15, JP2.16
- net +12V: no longer IC1.VI
- net 5V: now also JP2.11, JP2.12; no longer IC1.VO
- net GND: now also JP2.3, JP2.4, JP2.5, JP2.6, JP2.7, JP2.8; no longer IC1.GND, JP1.3, JP1.4, JP1.5, JP1.6, JP1.7, JP1.8
- net N$3: now also R62.2; no longer TR1.1
- net N$70: now also R62.1; no longer TR1.2, TR1.3
- net N$9: now also JP2.10, JP2.9; no longer JP1.10, JP1.9

Commit message: Reinstall
Parts:
- FADER1, FADER2, FADER3, FADER4, FADER5, FADER6, FADER7, FADER8: value 100k -> 50k
Changed lines of the file:
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@@
 <part name="C5" library="GMSN" deviceset="CAPACITOR_POL-US" device="153CLV-0505" value="10uF"/>
 <part name="GND8" library="GMSN" deviceset="GND" device=""/>
-<part name="FADER1" library="GMSN" deviceset="RESISTOR_VARIABLE_LED" device="" value="100k"/>
-<part name="FADER2" library="GMSN" deviceset="RESISTOR_VARIABLE_LED" device="" value="100k"/>
-<part name="FADER3" library="GMSN" deviceset="RESISTOR_VARIABLE_LED" device="" value="100k"/>
-<part name="FADER4" library="GMSN" deviceset="RESISTOR_VARIABLE_LED" device="" value="100k"/>
-<part name="FADER5" library="GMSN" deviceset="RESISTOR_VARIABLE_LED" device="" value="100k"/>
-<part name="FADER6" library="GMSN" deviceset="RESISTOR_VARIABLE_LED" device="" value="100k"/>
-<part name="FADER7" library="GMSN" deviceset="RESISTOR_VARIABLE_LED" device="" value="100k"/>
-<part name="FADER8" library="GMSN" deviceset="RESISTOR_VARIABLE_LED" device="" value="100k"/>
+<part name="FADER1" library="GMSN" deviceset="RESISTOR_VARIABLE_LED" device="" value="50k"/>
+<part name="FADER2" library="GMSN" deviceset="RESISTOR_VARIABLE_LED" device="" value="50k"/>
+<part name="FADER3" library="GMSN" deviceset="RESISTOR_VARIABLE_LED" device="" value="50k"/>
+<part name="FADER4" library="GMSN" deviceset="RESISTOR_VARIABLE_LED" device="" value="50k"/>
+<part name="FADER5" library="GMSN" deviceset="RESISTOR_VARIABLE_LED" device="" value="50k"/>
+<part name="FADER6" library="GMSN" deviceset="RESISTOR_VARIABLE_LED" device="" value="50k"/>
+<part name="FADER7" library="GMSN" deviceset="RESISTOR_VARIABLE_LED" device="" value="50k"/>
+<part name="FADER8" library="GMSN" deviceset="RESISTOR_VARIABLE_LED" device="" value="50k"/>
 <part name="GND4" library="GMSN" deviceset="GND" device=""/>
 <part name="IC6" library="GMSN" deviceset="MUX_1X8_CD4051" device="" value="CD4051"/>
